Commit message: dynamicArmExperiment

File: models/arm_2dof.urdf (robot description, URDF)
Before this commit: robot three_link_robot, 5 links, 4 joints
Joints:
- joint joint3: axis 0 0 1 -> (none); limit lower=-3.1416 upper=3.1416 effort=100 velocity=2.0 -> (none); type revolute -> fixed

File: models/arm_2dofIllusoryLengths.urdf (robot description, URDF)
Before this commit: robot three_link_robot, 5 links, 4 joints
Links:
- link link1: geometry collision cylinder length=0.315 radius=0.03; visual cylinder length=0.315 radius=0.03
- link link2: geometry collision cylinder length=0.410 radius=0.028; visual cylinder length=0.410 radius=0.028
- link link3: geometry collision cylinder length=0.395 radius=0.025; visual cylinder length=0.395 radius=0.025
Joints:
- joint ee_fixed_joint: origin xyz=0 0 0.390 rpy=0 0 0 -> xyz=0 0 0.395 rpy=0 0 0
- joint joint1: origin xyz=0 0 0.4 rpy=0 0 0 -> xyz=0 0 0.405 rpy=0 0 0
- joint joint2: origin xyz=0 0 0.310 rpy=0 0 0 -> xyz=0 0 0.315 rpy=0 0 0
- joint joint3: axis 0 0 1 -> (none); limit lower=-3.1416 upper=3.1416 effort=100 velocity=2.0 -> (none); type revolute -> fixed
