Commit message: archived experiment 1

File: models/arm_2dofIllusoryLengths.urdf (robot description, URDF)
Before this commit: robot two_link_robot, 5 links, 4 joints
Links:
- link link1: geometry collision cylinder length=0.31 radius=0.03; visual cylinder length=0.31 radius=0.03
- link link2: geometry collision cylinder length=0.401 radius=0.028; visual cylinder length=0.401 radius=0.028
- link link3: geometry collision cylinder length=0.391 radius=0.025; visual cylinder length=0.391 radius=0.025
Joints:
- joint ee_fixed_joint: origin xyz=0 0 0.395 rpy=0 0 0 -> xyz=0 0 0.391 rpy=0 0 0
- joint joint1: origin xyz=0 0 0.405 rpy=0 0 0 -> xyz=0 0 0.401 rpy=0 0 0
- joint joint2: origin xyz=0 0 0.315 rpy=0 0 0 -> xyz=0 0 0.31 rpy=0 0 0
