Commit message: updated Readme, changed model origins to align with paper

File: models/arm_3dof.urdf (robot description, URDF)
Before this commit: robot three_link_robot, 5 links, 4 joints
Joints:
- joint joint1: axis 0 1 0 -> 0 -1 0
- joint joint2: axis 0 1 0 -> 0 -1 0; origin xyz=0 0 0.310 rpy=0 0 0 -> xyz=0 0 0.310 rpy=0 1.57 0

File: models/arm_3dofLargeMass.urdf (robot description, URDF)
Before this commit: robot three_link_robot, 5 links, 4 joints
Joints:
- joint joint1: axis 0 1 0 -> 0 -1 0
- joint joint2: axis 0 1 0 -> 0 -1 0; origin xyz=0 0 0.310 rpy=0 0 0 -> xyz=0 0 0.310 rpy=0 1.57 0

File: models/arm_3dofMedMass.urdf (robot description, URDF)
Before this commit: robot three_link_robot, 5 links, 4 joints
Joints:
- joint joint1: axis 0 1 0 -> 0 -1 0
- joint joint2: axis 0 1 0 -> 0 -1 0; origin xyz=0 0 0.310 rpy=0 0 0 -> xyz=0 0 0.310 rpy=0 1.57 0

File: models/arm_3dofSmallMass.urdf (robot description, URDF)
Before this commit: robot three_link_robot, 5 links, 4 joints
Joints:
- joint joint1: axis 0 1 0 -> 0 -1 0
- joint joint2: axis 0 1 0 -> 0 -1 0; origin xyz=0 0 0.310 rpy=0 0 0 -> xyz=0 0 0.310 rpy=0 1.57 0
