Commit message: added a variety of experiments for the rbf cerebellum

File: experiments/experiments_02_thru_09/models/arm_3dof.urdf (robot description, URDF)
Before this commit: robot three_link_robot_illusion, 5 links, 4 joints
Links:
- link link1: geometry collision cylinder length=0.310 radius=0.03; visual cylinder length=0.310 radius=0.03
- link link2: geometry collision cylinder length=0.400 radius=0.028; visual cylinder length=0.400 radius=0.028
- link link3: geometry collision cylinder length=0.390 radius=0.025; visual cylinder length=0.390 radius=0.025
Joints:
- joint ee_fixed_joint: origin xyz=0 0 0.440 rpy=0 0 0 -> xyz=0 0 0.390 rpy=0 0 0
- joint joint1: origin xyz=0 0 0.450 rpy=0 0 0 -> xyz=0 0 0.4 rpy=0 0 0
- joint joint2: origin xyz=0 0 0.360 rpy=0 0 0 -> xyz=0 0 0.310 rpy=0 0 0

File: models/arm_2dofBigIllusoryMass.urdf (robot description, URDF)
Before this commit: robot three_link_robot_illusion, 5 links, 4 joints
Links:
- link ee_link: mass None -> 5.00; geometry collision sphere radius=0.03; visual sphere radius=0.03
- link link1: geometry collision cylinder length=0.310 radius=0.03; visual cylinder length=0.310 radius=0.03
- link link2: geometry collision cylinder length=0.400 radius=0.028; visual cylinder length=0.400 radius=0.028
- link link3: geometry collision cylinder length=0.390 radius=0.025; visual cylinder length=0.390 radius=0.025
Joints:
- joint ee_fixed_joint: origin xyz=0 0 0.440 rpy=0 0 0 -> xyz=0 0 0.390 rpy=0 0 0
- joint joint1: origin xyz=0 0 0.450 rpy=0 0 0 -> xyz=0 0 0.4 rpy=0 0 0
- joint joint2: origin xyz=0 0 0.360 rpy=0 0 0 -> xyz=0 0 0.310 rpy=0 0 0
- joint joint3: axis 0 0 1 -> (none); limit lower=-3.1416 upper=3.1416 effort=100 velocity=2.0 -> (none); type revolute -> fixed

File: models/arm_2dofIllusoryMass.urdf (robot description, URDF)
Before this commit: robot three_link_robot_illusion, 5 links, 4 joints
Links:
- link ee_link: mass None -> 0.500; geometry collision sphere radius=0.03; visual sphere radius=0.03
- link link1: geometry collision cylinder length=0.310 radius=0.03; visual cylinder length=0.310 radius=0.03
- link link2: geometry collision cylinder length=0.400 radius=0.028; visual cylinder length=0.400 radius=0.028
- link link3: geometry collision cylinder length=0.390 radius=0.025; visual cylinder length=0.390 radius=0.025
Joints:
- joint ee_fixed_joint: origin xyz=0 0 0.440 rpy=0 0 0 -> xyz=0 0 0.390 rpy=0 0 0
- joint joint1: origin xyz=0 0 0.450 rpy=0 0 0 -> xyz=0 0 0.4 rpy=0 0 0
- joint joint2: origin xyz=0 0 0.360 rpy=0 0 0 -> xyz=0 0 0.310 rpy=0 0 0
- joint joint3: axis 0 0 1 -> (none); limit lower=-3.1416 upper=3.1416 effort=100 velocity=2.0 -> (none); type revolute -> fixed

File: models/arm_3dofIllusoryMass.urdf (robot description, URDF)
Before this commit: robot three_link_robot_illusion, 5 links, 4 joints
Links:
- link ee_link: mass None -> 0.500; geometry collision sphere radius=0.03; visual sphere radius=0.03
- link link1: geometry collision cylinder length=0.310 radius=0.03; visual cylinder length=0.310 radius=0.03
- link link2: geometry collision cylinder length=0.400 radius=0.028; visual cylinder length=0.400 radius=0.028
- link link3: geometry collision cylinder length=0.390 radius=0.025; visual cylinder length=0.390 radius=0.025
Joints:
- joint ee_fixed_joint: origin xyz=0 0 0.440 rpy=0 0 0 -> xyz=0 0 0.390 rpy=0 0 0
- joint joint1: origin xyz=0 0 0.450 rpy=0 0 0 -> xyz=0 0 0.4 rpy=0 0 0
- joint joint2: origin xyz=0 0 0.360 rpy=0 0 0 -> xyz=0 0 0.310 rpy=0 0 0
